File: Hardware/_autosave-ATmegaXXM1_Breakout.kicad_pcb (KiCad board)
At the start: 2 copper layers, 57.1 x 50.2 mm, 37 parts, among them P1 VIN, P10 UART, P11 AREF, P12 Mounting Hole, P13 Mounting Hole, P14 Mounting Hole, P15 Mounting Hole, P2 PORTB, P3 PORTC, P4 PORTD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

Commit message: Changed routing & removed via in pad. Regenerated gerbers
Routing:
- net GND: track 356.9 -> 365.3 mm, vias 83 -> 84
- net /PB4: vias 5 -> 3
